File: pcb/rev.A/isa16_backplane.kicad_pcb (KiCad board)
At the start: 2 copper layers, 170.2 x 154.9 mm, 85 parts, among them J1 ATX-20, J2 Conn_01x02, J3 Conn_01x02, SW1 SW_Push, U1 74HCT14, U2 74HCT74, U3 7905

Commit message: update pcb rev.A files (final)
Parts:
- added H3: MountingHole_Pad, MountingHole:MountingHole_4mm_Pad_Via, F.Cu at (137.5, 121.1)
- added H4: MountingHole_Pad, MountingHole:MountingHole_4mm_Pad_Via, F.Cu at (292.5, 121.1)
- moved H10 3.05 mm to (292.5, 202.4)
- moved H9 3.05 mm to (137.5, 202.4)
- renumbered H8 to H10, H3 to H5, H4 to H6, H5 to H7, H6 to H8, H7 to H9
