File: pcb/rev.A/isa16_backplane.kicad_sch (KiCad schematic)
At the start: 85 parts, among them J1 ATX-20, J2 Conn_01x02, J3 Conn_01x02, SW1 SW_Push, U1 74HCT14, U2 74HCT74, U3 7905

Commit message: update pcb rev.A files (final)
Parts:
- added H3, H4: MountingHole_Pad, MountingHole:MountingHole_4mm_Pad_Via, symbol Mechanical:MountingHole_Pad
- renumbered H8 to H10, H3 to H5, H4 to H6, H5 to H7, H6 to H8, H7 to H9
Connections:
- net GND: now also H3.1, H4.1
Other:
- moved on the sheet: H1, H10, H2, H5, H6, H7, H8, H9
