File: pcb/rev.A1/isa16_backplane.kicad_pcb (KiCad board)
At the start: 2 copper layers, 170.2 x 154.9 mm, 87 parts, among them J1 ATX-20, J2 Conn_01x02, J3 Conn_01x02, SW1 SW_Push, U1 74HCT14, U2 74HCT74, U3 7905

Commit message: update pcb rev.A1 files (final)
Parts:
- J1: footprint my:Conn_Power_ATX_20pin_Alt -> my:Conn_Power_ATX_20pin_4.4mm
- SLOT1, SLOT2, SLOT3, SLOT4, SLOT5, SLOT6, SLOT7: footprint my:ISA16 -> my:ISA16_Slot
Other:
- board size 170.2 x 154.9 mm -> 171 x 155 mm
- board text added: "Layers: 2 Dimensions: 171x155mm Thickness: 1.6mm"
- board text removed: "Layers: 2 Dimensions: 170.18x154.94mm Thickness: 1.6mm"
