File: pcb/rev.A1/isa16_backplane.kicad_sch (KiCad schematic)
At the start: 87 parts, among them J1 ATX-20, J2 Conn_01x02, J3 Conn_01x02, SW1 SW_Push, U1 74HCT14, U2 74HCT74, U3 7905

Commit message: update pcb rev.A1 files (final)
Parts:
- J1: footprint my:Conn_Power_ATX_20pin_Alt -> my:Conn_Power_ATX_20pin_4.4mm
- SLOT1, SLOT2, SLOT3, SLOT4, SLOT5, SLOT6, SLOT7: footprint my:ISA16 -> my:ISA16_Slot
Changed lines of the file:
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@@
       (effects (font (size 1.27 1.27)))
     )
-    (property "Footprint" "my:ISA16" (at 53.34 100.33 0)
+    (property "Footprint" "my:ISA16_Slot" (at 53.34 100.33 0)
       (effects (font (size 1.27 1.27)) hide)
     )
@@
       (effects (font (size 1.27 1.27)))
     )
-    (property "Footprint" "my:ISA16" (at 134.62 100.33 0)
+    (property "Footprint" "my:ISA16_Slot" (at 134.62 100.33 0)
       (effects (font (size 1.27 1.27)) hide)
     )
@@
       (effects (font (size 1.27 1.27)))
     )
-    (property "Footprint" "my:ISA16" (at 215.9 100.33 0)
+    (property "Footprint" "my:ISA16_Slot" (at 215.9 100.33 0)
       (effects (font (size 1.27 1.27)) hide)
     )
@@
       (effects (font (size 1.27 1.27)))
     )
-    (property "Footprint" "my:ISA16" (at 297.18 100.33 0)
+    (property "Footprint" "my:ISA16_Slot" (at 297.18 100.33 0)
       (effects (font (size 1.27 1.27)) hide)
     )
@@
       (effects (font (size 1.27 1.27)))
     )
-    (property "Footprint" "my:ISA16" (at 378.46 100.33 0)
+    (property "Footprint" "my:ISA16_Slot" (at 378.46 100.33 0)
       (effects (font (size 1.27 1.27)) hide)
     )
@@
       (effects (font (size 1.27 1.27)))
     )
-    (property "Footprint" "my:ISA16" (at 541.02 99.06 0)
+    (property "Footprint" "my:ISA16_Slot" (at 541.02 99.06 0)
       (effects (font (size 1.27 1.27)) hide)
     )
@@
       (effects (font (size 1.27 1.27)))
     )
-    (property "Footprint" "my:ISA16" (at 459.74 99.06 0)
+    (property "Footprint" "my:ISA16_Slot" (at 459.74 99.06 0)
       (effects (font (size 1.27 1.27)) hide)
     )
@@
       (effects (font (size 1.27 1.27)))
     )
-    (property "Footprint" "my:Conn_Power_ATX_20pin_Alt" (at 106.68 215.9 0)
+    (property "Footprint" "my:Conn_Power_ATX_20pin_4.4mm" (at 106.68 215.9 0)
       (effects (font (size 1.27 1.27)) hide)
     )
